Commit message: feat : Add new camera link to support RGBD Camera and update plug-in for kinect

File: my_robot/urdf/my_robot.xacro (robot description, xacro)
@@ -196,4 +196,11 @@
             </visual>
         </link>
+        <link name="camera_link_optical">
+        </link>
+        <joint name="camera_optical_joint" type="fixed">
+          <origin xyz="0 0 0" rpy="-1.5707 0 -1.5707"/>
+          <parent link="camera"/>
+          <child link="camera_link_optical"/>
+        </joint>
         <joint name="hokuyo_joint" type="fixed">
             <origin xyz="0.15 0 0.1" rpy="0 0 0"/>
